File: models/KiCAD/fsr_array.kicad_pcb (KiCad board)
At the start: 4 copper layers, 100 x 100 mm, 94 parts, among them J1 scanning_ref1, J10 com_adc, J11 teensy_right, J12 teensy_left, J13 com_acc2, J14 com_acc1, J15 com_acc3, J16 com_acc4, J17 usb_B, J2 scanning_ref2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

Commit message: fixed minor bug + added ethernet teensy code
Parts:
- moved G*** 96.6 mm to (36.8, 115.5)
- moved G*** 87.1 mm to (52.0, 87.6)
- moved H1 36.6 mm to (69.8, 138.4)
- moved U$25 12.0 mm to (107.9, 143.5)
- moved U$61 9.94 mm to (196.8, 143.5)
- moved U$13 9.72 mm to (151.1, 143.5)
- moved U$29 9.68 mm to (153.6, 143.5)
- moved U$7 8.46 mm to (120.6, 140.9)
- moved U$1 8.44 mm to (140.9, 140.9)
- moved U$35 8.43 mm to (138.4, 140.9)
- moved U$23 8.43 mm to (130.8, 140.9)
- moved U$3 8.43 mm to (118.1, 140.9)
- moved U$5 8.42 mm to (143.5, 140.9)
- moved U$15 8.42 mm to (125.7, 140.9)
- moved U$11 8.42 mm to (123.2, 140.9)
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Connections:
- J11 pad 14: /SCK -> /SCLK
Routing:
- net /SCLK: track 40.3 -> 104.8 mm, vias 0 -> 1
- net /EOC2: track 73.9 -> 71.7 mm
- net Net-(ADC1-AIN12): track 17.7 -> 19.2 mm
- net Net-(ADC1-AIN14): track 20.4 -> 21.9 mm
- net Net-(ADC1-AIN8): track 22.6 -> 24.1 mm
- net Net-(ADC1-AIN10): track 18.7 -> 20.1 mm
- net Net-(ADC1-AIN6): track 27.3 -> 28.7 mm
- net Net-(ADC1-AIN2): track 38.4 -> 39.8 mm
- net Net-(ADC1-AIN4): track 32.6 -> 34.0 mm
- net Net-(ADC1-AIN5): track 29.9 -> 31.3 mm
- net Net-(ADC1-AIN9): track 20.8 -> 22.2 mm
- net Net-(ADC1-AIN3): track 35.7 -> 37.1 mm
- net Net-(ADC1-AIN1): track 41.6 -> 42.9 mm
- net Net-(ADC1-AIN0): track 44.2 -> 45.5 mm
- net Net-(ADC1-AIN7): track 24.8 -> 26.0 mm
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