File: models/LIS2DH_array/LIS2DH_array.kicad_pcb (KiCad board)
At the start: 2 copper layers, 113 x 113 mm, 82 parts, among them U1 LIS2DH12TR, U10 LIS2DH12TR, U11 LIS2DH12TR, U12 LIS2DH12TR, U13 LIS2DH12TR, U14 LIS2DH12TR, U15 LIS2DH12TR, U16 LIS2DH12TR, U17 SN74LVC1G32DCKR, U18 SN74LVC1G32DCKR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

Commit message: updated lis2dh arrays
Parts:
- C10, C12, C14, C16, C18, C2, C20, C22, C24, C26, C28, C30, C32, C4, C6, C8: value 1u -> 1uF
