File: models/customSquare16x16mini/customSquare16x16mini.kicad_pcb (KiCad board)
At the start: 2 copper layers, 60.5 x 42 mm, 4 parts, among them J1 Conn_01x16_Pin, J2 Conn_01x16_Pin

Commit message: updated
Routing:
- net /out0: track 71.2 -> 61.6 mm
- net /out1: track 66.4 -> 58.5 mm
- net /out2: track 62.6 -> 55.4 mm
- net /out3: track 58.9 -> 52.3 mm
- net /out4: track 55.2 -> 49.0 mm
- net /out5: track 51.5 -> 46.2 mm
- net /ain6: track 27.8 -> 33.0 mm
- net /out6: track 49.1 -> 43.9 mm
- net /ain9: track 27.8 -> 32.9 mm
- net /ain5: track 29.5 -> 34.5 mm
- net /ain10: track 29.5 -> 34.4 mm
- net /ain8: track 26.6 -> 31.5 mm
- net /ain7: track 26.6 -> 31.5 mm
- net /ain4: track 32.1 -> 36.9 mm
- net /ain11: track 32.2 -> 36.7 mm
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